File: kicad_files/sequencer.sch (KiCad schematic (older format))
At the start: 60 parts

Commit message: added midi ports, resistor on lcd cathode and access port for free pins
Parts:
- removed J?: DIN_5_FEMALE, symbol DIN_5_FEMALE
- removed R?: R, symbol R
- added D?: DIODE, symbol DIODE
- added P? (x3): DIN_5, symbol DIN_5
- added P?: CONN_02X05, symbol CONN_02X05
- added R? (x6): R, ~, symbol R
- added R?: R, symbol R
- added U?: PC900, symbol PC900
- added U?: 74LVC2G17GV, symbol 74LVC2G17GV
Connections:
- wire segments 260 -> 328
- no-connect marks 12 -> 18
Other:
- moved on the sheet: J?
